Commit message: Add files via upload

File: battlebot_spinner/urdf/spinner_bot.xacro (robot description, xacro)
@@ -1,48 +1,167 @@
-<!-- urdf/spinner_bot.xacro -->
-<robot xmlns:xacro="http://ros.org/wiki/xacro" name="spinner_bot">
-  <link name="world"/> <joint name="world_to_base_link_fixed_joint" type="fixed">
-    <parent link="world"/>
-    <child link="base_link"/>
-    <origin xyz="0 0 0" rpy="0 0 0"/>
-  </joint>
+<?xml version="1.0"?>
+<robot xmlns:xacro="http://www.ros.org/wiki/xacro" name="battlebot">
+  <xacro:property name="PI" value="3.1415926535897931"/>
+  <xacro:property name="chassis_mass" value="5.0"/>
+  <xacro:property name="wheel_mass" value="0.5"/>
+  <xacro:property name="weapon_mass" value="1.5"/>
+  <xacro:property name="wheel_radius" value="0.1"/>
+  <xacro:property name="chassis_width" value="0.4"/>
+  <xacro:property name="chassis_length" value="0.6"/>
+  <xacro:property name="chassis_height" value="0.1"/>
+  <xacro:property name="weapon_radius" value="0.15"/>
+  <xacro:property name="weapon_thickness" value="0.02"/>
+  <material name="red">
+    <color rgba="1.0 0.0 0.0 1.0"/>
+  </material>
+  <material name="silver">
+    <color rgba="0.8 0.8 0.8 1.0"/>
+  </material>
+  <material name="black">
+    <color rgba="0.1 0.1 0.1 1.0"/>
+  </material>
   <link name="base_link">
+    <inertial>
+      <mass value="${chassis_mass}"/>
+      <origin xyz="0 0 0" rpy="0 0 0"/>
+      <inertia ixx="${chassis_mass/12.0 * (chassis_height*chassis_height + chassis_width*chassis_width)}"
+               ixy="0.0" ixz="0.0"
+               iyy="${chassis_mass/12.0 * (chassis_length*chassis_length + chassis_height*chassis_height)}"
+               iyz="0.0"
+               izz="${chassis_mass/12.0 * (chassis_length*chassis_length + chassis_width*chassis_width)}"/>
+    </inertial>
+    <collision>
+      <geometry>
+        <box size="${chassis_length} ${chassis_width} ${chassis_height}"/>
+      </geometry>
+    </collision>
     <visual>
       <geometry>
-        <box size="0.5 0.5 0.2"/>
+        <box size="${chassis_length} ${chassis_width} ${chassis_height}"/>
       </geometry>
+      <material name="red"/>
     </visual>
+  </link>
+  <link name="right_wheel">
+    <inertial>
+      <mass value="${wheel_mass}"/>
+      <origin xyz="0 0 0" rpy="${PI/2} 0 0"/>
+      <inertia ixx="${wheel_mass * wheel_radius * wheel_radius / 2.0}"
+               ixy="0.0" ixz="0.0"
+               iyy="${wheel_mass * wheel_radius * wheel_radius / 2.0}"
+               iyz="0.0"
+               izz="${wheel_mass * wheel_radius * wheel_radius}"/>
+    </inertial>
+    <collision>
+      <origin xyz="0 0 0" rpy="${PI/2} 0 0"/>
+      <geometry>
+        <cylinder radius="${wheel_radius}" length="0.05"/>
+      </geometry>
+    </collision>
+    <visual>
+      <origin xyz="0 0 0" rpy="${PI/2} 0 0"/>
+      <geometry>
+        <cylinder radius="${wheel_radius}" length="0.05"/>
+      </geometry>
+      <material name="black"/>
+    </visual>
+  </link>
+  <link name="left_wheel">
+    <inertial>
+      <mass value="${wheel_mass}"/>
+      <origin xyz="0 0 0" rpy="${PI/2} 0 0"/>
+      <inertia ixx="${wheel_mass * wheel_radius * wheel_radius / 2.0}"
+               ixy="0.0" ixz="0.0"
+               iyy="${wheel_mass * wheel_radius * wheel_radius / 2.0}"
+               iyz="0.0"
+               izz="${wheel_mass * wheel_radius * wheel_radius}"/>
+    </inertial>
+    <collision>
+      <origin xyz="0 0 0" rpy="${PI/2} 0 0"/>
+      <geometry>
+        <cylinder radius="${wheel_radius}" length="0.05"/>
+      </geometry>
+    </collision>
+    <visual>
+      <origin xyz="0 0 0" rpy="${PI/2} 0 0"/>
+      <geometry>
+        <cylinder radius="${wheel_radius}" length="0.05"/>
+      </geometry>
+      <material name="black"/>
+    </visual>
+  </link>
+  <link name="weapon">
+    <inertial>
+      <mass value="${weapon_mass}"/>
+      <origin xyz="0 0 0" rpy="0 0 0"/>
+      <inertia ixx="${weapon_mass * (3*weapon_radius*weapon_radius + weapon_thickness*weapon_thickness) / 12.0}"
+               ixy="0.0" ixz="0.0"
+               iyy="${weapon_mass * (3*weapon_radius*weapon_radius + weapon_thickness*weapon_thickness) / 12.0}"
+               iyz="0.0"
+               izz="${weapon_mass * weapon_radius * weapon_radius / 2.0}"/>
+    </inertial>
     <collision>
       <geometry>
-        <box size="0.5 0.5 0.2"/>
+        <cylinder radius="${weapon_radius}" length="${weapon_thickness}"/>
       </geometry>
     </collision>
-    <inertial>
-      <mass value="5.0"/>
-      <inertia ixx="0.1" iyy="0.1" izz="0.1" ixy="0.0" ixz="0.0" iyz="0.0"/>
-    </inertial>
-  </link>
-  <!-- Spinner Weapon -->
-  <link name="spinner">
     <visual>
       <geometry>
-        <cylinder length="0.02" radius="0.3"/>
+        <cylinder radius="${weapon_radius}" length="${weapon_thickness}"/>
       </geometry>
+      <material name="silver"/>
     </visual>
-    <collision>
-      <geometry>
-        <cylinder length="0.02" radius="0.3"/>
-      </geometry>
-    </collision>
-    <inertial>
-      <mass value="1.0"/>
-      <inertia ixx="0.02" iyy="0.02" izz="0.01" ixy="0.0" ixz="0.0" iyz="0.0"/>
-    </inertial>
   </link>
-  <joint name="spinner_joint" type="continuous">
+  <joint name="right_wheel_joint" type="continuous">
     <parent link="base_link"/>
-    <child link="spinner"/>
-    <origin xyz="0 0 0.11" rpy="0 0 0"/>
+    <child link="right_wheel"/>
+    <origin xyz="0 -${chassis_width/2 + 0.02} 0" rpy="0 0 0"/>
+    <axis xyz="0 1 0"/>
+    <dynamics damping="0.1" friction="0.1"/>
+  </joint>
+  <joint name="left_wheel_joint" type="continuous">
+    <parent link="base_link"/>
+    <child link="left_wheel"/>
+    <origin xyz="0 ${chassis_width/2 + 0.02} 0" rpy="0 0 0"/>
+    <axis xyz="0 1 0"/>
+    <dynamics damping="0.1" friction="0.1"/>
+  </joint>
+  <joint name="weapon_joint" type="continuous">
+    <parent link="base_link"/>
+    <child link="weapon"/>
+    <origin xyz="${chassis_length/2 - weapon_radius/2} 0 ${chassis_height/2 + weapon_thickness/2}" rpy="0 0 0"/>
     <axis xyz="0 0 1"/>
-    <limit effort="5.0" velocity="10.0"/>
+    <dynamics damping="0.01" friction="0.01"/>
   </joint>
+  <gazebo>
+    <plugin name="differential_drive_controller" filename="libgazebo_ros_diff_drive.so">
+      <updateRate>100</updateRate>
+      <leftJoint>left_wheel_joint</leftJoint>
+      <rightJoint>right_wheel_joint</rightJoint>
+      <wheelSeparation>${chassis_width + 0.04}</wheelSeparation>
+      <wheelDiameter>${2 * wheel_radius}</wheelDiameter>
+      <wheelAcceleration>1.0</wheelAcceleration>
+      <wheelTorque>20</wheelTorque>
+      <commandTopic>cmd_vel</commandTopic>
+      <odometryTopic>odom</odometryTopic>
+      <odometryFrame>odom</odometryFrame>
+      <robotBaseFrame>base_link</robotBaseFrame>
+      <publishOdomTF>true</publishOdomTF>
+      <publishWheelTF>false</publishWheelTF>
+      <odometrySource>world</odometrySource>
+      <publishTf>true</publishTf>
+    </plugin>
+  </gazebo>
+  <gazebo>
+    <plugin name="weapon_controller" filename="libgazebo_ros_joint_state_publisher.so">
+      <jointName>weapon_joint</jointName>
+      <updateRate>100</updateRate>
+    </plugin>
+  </gazebo>
+  <gazebo>
+    <plugin name="weapon_motor" filename="libgazebo_ros_joint_motor.so">
+      <joint>weapon_joint</joint>
+      <topic>weapon_speed</topic>
+      <jointType>velocity</jointType>
+    </plugin>
+  </gazebo>
 </robot>
