Commit message: Added new feature

File: urdf/battlebot_2.urdf (robot description, URDF)
Before this commit: robot battlebot_2, 5 links, 4 joints
Links:
- removed link saw_link
- added link ${frame_prefix}saw_link, mass 0.75; collision mesh filename=model://saw_blade_1/meshes/Sawblade.dae scale=2.01 2.01 1.01; visual mesh filename=model://saw_blade_1/meshes/Sawblade.dae scale=2 2 1

Commit message: Added new feature

File: urdf/battlebot_2.urdf (robot description, URDF)
Before this commit: robot battlebot_2, 5 links, 4 joints
Links:
- removed link ${frame_prefix}saw_link
- added link saw_link, mass 0.6; collision cylinder length=0.02 radius=0.2; visual cylinder length=0.02 radius=0.2
