Commit message: Added new feature

File: urdf/battlebot_1.urdf (robot description, URDF)
Before this commit: robot battlebot_1, 5 links, 4 joints
Links:
- removed link contact_sensor_link
- link left_wheel: mass 1.5 -> 3
- link right_wheel: mass 1.5 -> 3
- link saw_link: mass 0.6 -> 1; geometry collision cylinder length=0.02 radius=0.55; visual mesh filename=model://saw_blade_1/meshes/Sawblade.dae scale=2 2 1
Joints:
- removed joint contact_sensor_joint
- joint left_wheel_joint: origin xyz=0 0.45 0.1 rpy=0 0 0 -> xyz=0 0.45 0.18 rpy=0 0 0
- joint right_wheel_joint: origin xyz=0 -0.45 0.1 rpy=0 0 0 -> xyz=0 -0.45 0.18 rpy=0 0 0
- joint saw_joint: axis (none) -> 1 0 0

File: urdf/battlebot_2.urdf (robot description, URDF)
Before this commit: robot battlebot_2, 5 links, 4 joints
Links:
- removed link contact_sensor_link
- link left_wheel: mass 1.5 -> 3
- link right_wheel: mass 1.5 -> 3
- link saw_link: mass 0.6 -> 1; geometry collision cylinder length=0.02 radius=0.55; visual mesh filename=model://saw_blade_1/meshes/Sawblade.dae scale=2 2 1
Joints:
- removed joint contact_sensor_joint
- joint left_wheel_joint: origin xyz=0 0.45 0.1 rpy=0 0 0 -> xyz=0 0.45 0.18 rpy=0 0 0
- joint right_wheel_joint: origin xyz=0 -0.45 0.1 rpy=0 0 0 -> xyz=0 -0.45 0.18 rpy=0 0 0
- joint saw_joint: axis (none) -> 1 0 0

Commit message: Added new feature

File: urdf/battlebot_1.urdf (robot description, URDF)
Before this commit: robot battlebot_1, 4 links, 3 joints
Links:
- removed link left_wheel
- removed link right_wheel
- removed link saw_link
- added link left_wheel_link, mass 1.0; collision cylinder length=0.05 radius=0.15; visual cylinder length=0.05 radius=0.15
- added link right_wheel_link, mass 1.0; collision cylinder length=0.05 radius=0.15; visual cylinder length=0.05 radius=0.15
- link base_link: mass 15.0 -> 10.0; geometry collision box size=0.8 0.5 0.2; visual box size=0.8 0.5 0.2
Joints:
- removed joint saw_joint
- joint left_wheel_joint: child left_wheel -> left_wheel_link; origin xyz=0 0.45 0.18 rpy=0 0 0 -> xyz=0.0 0.275 0 rpy=0 0 0
- joint right_wheel_joint: child right_wheel -> right_wheel_link; origin xyz=0 -0.45 0.18 rpy=0 0 0 -> xyz=0.0 -0.275 0 rpy=0 0 0

File: urdf/battlebot_2.urdf (robot description, URDF)
Before this commit: robot battlebot_2, 4 links, 3 joints
Links:
- removed link left_wheel
- removed link right_wheel
- removed link saw_link
- added link left_wheel_link, mass 1.0; collision cylinder length=0.05 radius=0.15; visual cylinder length=0.05 radius=0.15
- added link right_wheel_link, mass 1.0; collision cylinder length=0.05 radius=0.15; visual cylinder length=0.05 radius=0.15
- link base_link: mass 15.0 -> 10.0; geometry collision box size=0.8 0.5 0.2; visual box size=0.8 0.5 0.2
Joints:
- removed joint saw_joint
- joint left_wheel_joint: child left_wheel -> left_wheel_link; origin xyz=0 0.45 0.18 rpy=0 0 0 -> xyz=0.0 0.275 0 rpy=0 0 0
- joint right_wheel_joint: child right_wheel -> right_wheel_link; origin xyz=0 -0.45 0.18 rpy=0 0 0 -> xyz=0.0 -0.275 0 rpy=0 0 0

Commit message: Added new feature

File: urdf/battlebot_1.urdf (robot description, URDF)
Before this commit: robot battlebot_1, 3 links, 2 joints
Links:
- link base_link: mass 10.0 -> 15.0; geometry collision box size=1.3 0.9 0.3; visual box size=1.3 0.9 0.3
- link left_wheel_link: geometry collision cylinder length=0.1 radius=0.24; visual cylinder length=0.1 radius=0.24
- link right_wheel_link: geometry collision cylinder length=0.1 radius=0.24; visual cylinder length=0.1 radius=0.24
Joints:
- joint left_wheel_joint: origin xyz=0.0 0.275 0 rpy=0 0 0 -> xyz=0.0 0.525 0.2 rpy=0 0 0
- joint right_wheel_joint: origin xyz=0.0 -0.275 0 rpy=0 0 0 -> xyz=0.0 -0.525 0.2 rpy=0 0 0

File: urdf/battlebot_2.urdf (robot description, URDF)
Before this commit: robot battlebot_2, 3 links, 2 joints
Links:
- link base_link: mass 10.0 -> 15.0; geometry collision box size=1.3 0.9 0.3; visual box size=1.3 0.9 0.3
- link left_wheel_link: geometry collision cylinder length=0.1 radius=0.24; visual cylinder length=0.1 radius=0.24
- link right_wheel_link: geometry collision cylinder length=0.1 radius=0.24; visual cylinder length=0.1 radius=0.24
Joints:
- joint left_wheel_joint: origin xyz=0.0 0.275 0 rpy=0 0 0 -> xyz=0.0 0.525 0.2 rpy=0 0 0
- joint right_wheel_joint: origin xyz=0.0 -0.275 0 rpy=0 0 0 -> xyz=0.0 -0.525 0.2 rpy=0 0 0
